File: 电路/主控器/PM_Controller_R1/PM_Controller.kicad_pcb (KiCad board)
At the start: 4 copper layers, 90 x 61.5 mm, 132 parts, among them J1 Conn_01x04_Socket, J10 Conn_02x04_Odd_Even, J11 Conn_02x06_Odd_Even, J2 Conn_01x04_Socket, J3 Conn_01x04_Socket, J4 Conn_01x04_Socket, J5 Conn_01x02_Pin, J6 Conn_01x02_Pin, J7 Conn_02x04_Odd_Even, J8 Conn_01x04_Pin, J9 Conn_01x04_Socket, P2V5 SolderJumper_2_Open, P3V3 SolderJumper_2_Open, Q1 AO3401A, Q2 AO3400A, Q3 AO3400A, Q4 AO3400A, Q5 AO3400A, Q6 AO3400A, U1 AT24CS08-SSHM, U10 TMP102xxDRL, U11 TPS2552DDBVR, U12 TLP127, U13 TLV61048DBVR, U2 AMS1117-3.3, U3 STM32G431RBTx, U5 BQ21040DBV, U6 TPS2552DDBVR, U7 STM32L011D4Px, U8 ME6211C25M5, U9 AT24CS08-SSHM, Y1 32.768kHz, Y2 24Mhz

Commit message: ZUI init
Parts:
- removed C39: 22uf, Capacitor_Tantalum_SMD:CP_EIA-3528-21_Kemet-B_HandSolder
- removed C40: 1uf, Capacitor_SMD:C_1206_3216Metric_Pad1.33x1.80mm_HandSolder
- removed C41: 10uf, Capacitor_SMD:C_1206_3216Metric_Pad1.33x1.80mm_HandSolder
- removed D4: 1N5819WS, Diode_SMD:D_SOD-323_HandSoldering
- removed R43: 330k, Resistor_SMD:R_0603_1608Metric_Pad0.98x0.95mm_HandSolder
- removed R44: 51k, Resistor_SMD:R_0603_1608Metric_Pad0.98x0.95mm_HandSolder
- removed R45: 10k, Resistor_SMD:R_0603_1608Metric_Pad0.98x0.95mm_HandSolder
- removed U13: TLV61048DBVR, footprints:SOT-23-6_DBV_TEX
- added C13: 22uf, Capacitor_SMD:C_0603_1608Metric_Pad1.08x0.95mm_HandSolder, F.Cu at (53.4, 149.0)
- added C15: 100nf, Capacitor_SMD:C_0603_1608Metric_Pad1.08x0.95mm_HandSolder, F.Cu at (53.4, 152.4)
- added C16: 820pf, Capacitor_SMD:C_0603_1608Metric_Pad1.08x0.95mm_HandSolder, F.Cu at (53.4, 158.5)
- added C4: 22uf, Capacitor_Tantalum_SMD:CP_EIA-3528-21_Kemet-B_Pad1.50x2.35mm_HandSolder, F.Cu at (61.9, 154.5)
- added C9: 1uf, Capacitor_SMD:C_0603_1608Metric_Pad1.08x0.95mm_HandSolder, F.Cu at (53.4, 150.5)
- added D1: SS32, Diode_SMD:D_SMA_Handsoldering, F.Cu at (61.9, 149.5)
- added R10: 82k, Resistor_SMD:R_0603_1608Metric_Pad0.98x0.95mm_HandSolder, B.Cu at (55.8, 156.8)
- added R11: 27k, Resistor_SMD:R_0603_1608Metric_Pad0.98x0.95mm_HandSolder, B.Cu at (54.3, 156.8)
- added R9: 56.2k, Resistor_SMD:R_0603_1608Metric_Pad0.98x0.95mm_HandSolder, F.Cu at (53.4, 157.0)
- added U4: TPS61085DGK, Package_SO:VSSOP-8_3x3mm_P0.65mm, F.Cu at (56.9, 154.5)
- J5: footprint Connector_Wire:SolderWire-0.5sqmm_1x02_P4.8mm_D0.9mm_OD2.3mm -> Connector_Wire:SolderWire-0.1sqmm_1x02_P3.6mm_D0.4mm_OD1mm_Relief
- L1: footprint Inductor_SMD:L_APV_APH0650 -> Inductor_SMD:L_APV_ANR5040
- moved L1 7.21 mm to (56.4, 145.0), turned to 0 degrees
- moved J5 6.00 mm to (58.9, 140.8), turned to 90 degrees
- moved R25 2.21 mm to (66.5, 146.2)
- moved C11 1.17 mm to (58.2, 155.0)
- moved R23 0.45 mm to (62.0, 142.5), turned to 90 degrees
- moved R24 0.45 mm to (63.5, 142.5)
- moved C6 0.15 mm to (66.9, 159.9)
Routing:
- net /BAT_OUT: track 5.81 -> 28.0 mm, vias 5 -> 2
- net Net-(U13-FB): track 5.83 -> 0.00 mm
- net Net-(U4-FB): track 0.00 -> 5.30 mm, vias 0 -> 1
- net Net-(D1-A): track 1.46 -> 6.27 mm
- net Net-(U4-SS): track 0.00 -> 4.29 mm
- net /VBAT5: track 3.78 -> 7.26 mm, vias 0 -> 1
- net Net-(U13-EN): track 3.23 -> 0.00 mm
- net Net-(C16-Pad2): track 0.00 -> 2.40 mm
- net /ADC1_15: track 31.9 -> 34.2 mm
- net Net-(U4-COMP): track 0.00 -> 1.77 mm
- net Net-(R23-Pad1): track 7.22 -> 5.63 mm
- net GND: track 101.7 -> 101.2 mm, vias 102 -> 100
- net +BATT: vias 9 -> 10
- added copper zone on F.Cu, net Net-(U4-SS)
Other:
- outline, holes or cut-outs redrawn
