File: 电路/主控器/PM_Controller_R1/PM_Controller.kicad_sch (KiCad schematic)
At the start: 132 parts, among them J1 Conn_01x04_Socket, J10 Conn_02x04_Odd_Even, J11 Conn_02x06_Odd_Even, J2 Conn_01x04_Socket, J3 Conn_01x04_Socket, J4 Conn_01x04_Socket, J5 Conn_01x02_Pin, J6 Conn_01x02_Pin, J7 Conn_02x04_Odd_Even, J8 Conn_01x04_Pin, J9 Conn_01x04_Socket, P2V5 SolderJumper_2_Open, P3V3 SolderJumper_2_Open, Q1 AO3401A, Q2 AO3400A, Q3 AO3400A, Q4 AO3400A, Q5 AO3400A, Q6 AO3400A, U1 AT24CS08-SSHM, U10 TMP102xxDRL, U11 TPS2552DDBVR, U12 TLP127, U13 TLV61048DBVR, U2 AMS1117-3.3, U3 STM32G431RBTx, U5 BQ21040DBV, U6 TPS2552DDBVR, U7 STM32L011D4Px, U8 ME6211C25M5, U9 AT24CS08-SSHM, Y1 32.768kHz, Y2 24Mhz

Commit message: ZUI init
Parts:
- removed C39: 22uf, Capacitor_Tantalum_SMD:CP_EIA-3528-21_Kemet-B_HandSolder, symbol Device:C_Polarized
- removed C40: 1uf, Capacitor_SMD:C_1206_3216Metric_Pad1.33x1.80mm_HandSolder, symbol Device:C
- removed C41: 10uf, Capacitor_SMD:C_1206_3216Metric_Pad1.33x1.80mm_HandSolder, symbol Device:C
- removed D4: 1N5819WS, Diode_SMD:D_SOD-323_HandSoldering, symbol Diode:1N5819WS
- removed R43: 150k, Resistor_SMD:R_0603_1608Metric_Pad0.98x0.95mm_HandSolder, symbol Device:R
- removed R44: 33k, Resistor_SMD:R_0603_1608Metric_Pad0.98x0.95mm_HandSolder, symbol Device:R
- removed R45: 10k, Resistor_SMD:R_0603_1608Metric_Pad0.98x0.95mm_HandSolder, symbol Device:R
- removed U13: TLV61048DBVR, SOT-23-6_DBV_TEX, symbol 2025-04-10_12-12-53:TLV61048DBVR
- added C13: 22uf, Capacitor_SMD:C_0603_1608Metric_Pad1.08x0.95mm_HandSolder, symbol Device:C
- added C15: 100nf, Capacitor_SMD:C_0603_1608Metric_Pad1.08x0.95mm_HandSolder, symbol Device:C
- added C16: 820pf, Capacitor_SMD:C_0603_1608Metric_Pad1.08x0.95mm_HandSolder, symbol Device:C
- added C4: 22uf, Capacitor_Tantalum_SMD:CP_EIA-3528-21_Kemet-B_Pad1.50x2.35mm_HandSolder, symbol Device:C_Polarized
- added C9: 1uf, Capacitor_SMD:C_0603_1608Metric_Pad1.08x0.95mm_HandSolder, symbol Device:C
- added D1: SS32, Diode_SMD:D_SMA_Handsoldering, symbol Diode:SS32
- added R10: 82k, Resistor_SMD:R_0603_1608Metric_Pad0.98x0.95mm_HandSolder, symbol Device:R
- added R11: 27k, Resistor_SMD:R_0603_1608Metric_Pad0.98x0.95mm_HandSolder, symbol Device:R
- added R9: 56.2k, Resistor_SMD:R_0603_1608Metric_Pad0.98x0.95mm_HandSolder, symbol Device:R
- added U4: TPS61085DGK, Package_SO:VSSOP-8_3x3mm_P0.65mm, symbol Regulator_Switching:TPS61085DGK
- J5: footprint Connector_Wire:SolderWire-0.5sqmm_1x02_P4.8mm_D0.9mm_OD2.3mm -> Connector_Wire:SolderWire-0.1sqmm_1x02_P3.6mm_D0.4mm_OD1mm_Relief
- L1: footprint Inductor_SMD:L_APV_APH0650 -> Inductor_SMD:L_APV_ANR5040
Connections:
- net BAT_OUT: now also C13.1, C9.1, U4.3 (EN), U4.6 (VIN), U4.7 (FREQ)
- net GND: now also C13.2, C15.1, C16.1, C4.2, C9.2, R11.1, U4.4 (GND)
- net VBAT5: now also C4.1, D1.1 (K), R10.2
- net at L1.2: now also D1.2 (A), U4.5 (SW)
- new net: R9.1, U4.1 (COMP)
- new net: C16.2, R9.2
- new net: C15.2, U4.8 (SS)
- new net: R10.1, R11.2, U4.2 (FB)
- no-connect marks 12 -> 11
